Commit message: 移除相機

File: src/ardrone_simulator_gazebo7/cvg_sim_gazebo/urdf/quadrotor_base.urdf (copy).xacro (robot description, xacro)
@@ -38,6 +38,35 @@
           <child link="${prefix}_dummy_link"/>
     </joint>
+    <link name='${prefix}_link_0'>
+	    <inertial>
+	     <origin xyz="0 0 0.5" rpy="0 0 0"/>
+	     <mass value="0.00000"/>
+	     <inertia ixx="0"  ixy="0"  ixz="0" iyy="0" iyz="0" izz="0" />
+	   </inertial>
+	   <visual>
+	     <origin xyz="-0.3 0 0" rpy="0 0 0" />
+	     <geometry>
+	       <box size="0.01 0.6 0.3" />
+	     </geometry>
+     <material name="Cyan">
+       <color rgba="0 1.0 1.0 1.0"/>
+     </material>
+	   </visual>
+	   <collision>
+	     <origin xyz="0 0 0" rpy="0 0 0"/>
+	     <geometry>
+	       <box size="0.01 0.1 0.1" />
+	     </geometry>
+	   </collision>
+    </link>
+    <joint name="${prefix}_marker_joint" type="fixed">
+ 	        <parent link="${prefix}_base_link"/>
+          <child link='${prefix}_link_0'/>
+    </joint>
     <gazebo reference="${prefix}_base_link">
       <turnGravityOff>false</turnGravityOff>
+    </gazebo>
+    <gazebo reference="${prefix}_link_0">
+        <material value="RepeatedTexture${markerNO}"/>
     </gazebo>
     <!-- Gazebo Plugins -->

File: src/ardrone_simulator_gazebo7/cvg_sim_gazebo/urdf/quadrotor_with_sensors.urdf.xacro (robot description, xacro)
@@ -24,8 +24,8 @@
     <!-- The following two cameras should be united to one! -->
     <!-- Forward facing camera -->
-    <xacro:include filename="$(find cvg_sim_gazebo)/urdf/sensors/generic_camera.urdf.xacro" />
+    <!-- <xacro:include filename="$(find cvg_sim_gazebo)/urdf/sensors/generic_camera.urdf.xacro" />
     <xacro:generic_camera name="front" sim_name="ardrone" parent="$(arg prefix)_base_link" update_rate="30" res_x="960" res_y="720" image_format="R8G8B8" hfov="${81*M_PI/180}">
       <origin xyz="0.21 0.0 0.01" rpy="0 0 0"/>
-    </xacro:generic_camera>
+    </xacro:generic_camera> -->
     <!-- Downward facing camera
     <xacro:include filename="$(find cvg_sim_gazebo)/urdf/sensors/generic_camera.urdf.xacro" />
